File: 2890/pcbs/pico_cartridge/pico_cartridge_2890/pico_cartridge_2890.kicad_pcb (KiCad board)
At the start: 2 copper layers, 58.6 x 138 mm, 41 parts, among them J2 monroe-2890-cart-conn, J5 Conn_01x04_Female, SW1 A, SW2 A, SW7 A

Commit message: "Update"
Parts:
- moved R28 30.4 mm to (89.0, 152.5)
- moved R7 25.6 mm to (117.0, 152.5)
- moved R8 25.3 mm to (91.5, 152.5)
- moved R11 21.2 mm to (114.5, 152.5)
- moved R6 17.8 mm to (94.0, 152.7)
- moved R23 16.1 mm to (96.5, 152.5)
- moved R18 15.5 mm to (112.0, 152.5)
- moved R12 11.5 mm to (99.0, 152.5)
- moved R13 9.94 mm to (109.0, 152.5), turned to -90 degrees
- moved R15 7.18 mm to (106.5, 152.5)
- moved R5 0.30 mm to (117.0, 157.5)
- moved R24 0.22 mm to (104.0, 152.5)
Connections:
- J2 pad 16: unconnected-(J2-Pin_16-Pad16) -> Net-(J2-Pin_16)
- J2 pad 2: +5V -> unconnected-(J2-Pin_2-Pad2)
- J2 pad 20: Net-(J2-Pin_20) -> unconnected-(J2-Pin_20-Pad20)
- J2 pad 30: unconnected-(J2-Pin_30-Pad30) -> Net-(J2-Pin_30)
- J2 pad 32: unconnected-(J2-Pin_32-Pad32) -> GND
- J2 pad 34: unconnected-(J2-Pin_34-Pad34) -> +5V
- J2 pad 4: GND -> unconnected-(J2-Pin_4-Pad4)
- J2 pad 6: Net-(J2-Pin_6) -> unconnected-(J2-Pin_6-Pad6)
- R11 pad 2: Net-(J2-Pin_26) -> Net-(J2-Pin_10)
- R12 pad 2: Net-(J2-Pin_14) -> Net-(J2-Pin_22)
- R13 pad 2: Net-(J2-Pin_22) -> Net-(J2-Pin_14)
- R15 pad 2: Net-(J2-Pin_20) -> Net-(J2-Pin_16)
- R18 pad 2: Net-(J2-Pin_24) -> Net-(J2-Pin_12)
- R23 pad 2: Net-(J2-Pin_12) -> Net-(J2-Pin_24)
- R28 pad 2: Net-(J2-Pin_6) -> Net-(J2-Pin_30)
- R6 pad 2: Net-(J2-Pin_10) -> Net-(J2-Pin_26)
- R7 pad 2: Net-(J2-Pin_28) -> Net-(J2-Pin_8)
- R8 pad 2: Net-(J2-Pin_8) -> Net-(J2-Pin_28)
Routing:
- net GPIO0: track 139.0 -> 109.5 mm
- net CEOE2: track 105.7 -> 85.0 mm
- net Net-(J2-Pin_6): track 17.9 -> 0.00 mm, vias 1 -> 0
- net Net-(J2-Pin_16): track 0.00 -> 17.9 mm, vias 0 -> 1
- net Net-(J2-Pin_30): track 0.00 -> 17.6 mm, vias 0 -> 1
- net GPIO1: track 112.8 -> 129.0 mm, vias 1 -> 3
- net GPIO32: track 112.0 -> 125.7 mm, vias 1 -> 3
- net +5V: track 95.4 -> 82.2 mm, vias 3 -> 5
- net Net-(J2-Pin_20): track 12.3 -> 0.00 mm, vias 1 -> 0
- net GPIO33: track 113.8 -> 120.7 mm, vias 1 -> 5
- net GPIO6: track 106.0 -> 112.1 mm, vias 3 -> 5
- net Net-(J2-Pin_14): track 11.7 -> 16.8 mm
- net Net-(J2-Pin_12): track 12.1 -> 17.0 mm
- net Net-(J2-Pin_26): track 12.5 -> 17.0 mm
- net GPIO38: track 102.8 -> 106.5 mm, vias 1 -> 3
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Other:
- board text added: "Monroe 2890 Pico cartridge V1.1 April 2026 menadue@gmail.com"
- board text removed: "Monroe 2890 Pico cartridge V1.0 March 2026 menadue@gmail.com"
